Commit message: added mesh files for fetch head and modified fetch.urdf

File: fetch_description/robots/fetch.urdf (robot description, URDF)
Before this commit: robot fetch, 26 links, 25 joints
Links:
- added link head_box_link, mass 2.2556; collision mesh filename=package://fetch_description/meshes/head_box_link_collision.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; visual mesh filename=package://fetch_description/meshes/head_box_link.dae
- added link t265_base_link
Joints:
- added joint head_box_joint: type fixed, parent head_pan_link, child head_box_link, origin xyz=0 0 0 rpy=0 0 0
- added joint t265_joint: type fixed, parent head_pan_link, child t265_base_link, origin xyz=0 0 0 rpy=0.145426 0.00775 0.16

Commit message: fixed scale of fetch head box meshes in urdf

File: fetch_description/robots/fetch.urdf (robot description, URDF)
Before this commit: robot fetch, 28 links, 27 joints
Links:
- link head_box_link: geometry collision mesh filename=package://fetch_description/meshes/head_box_link_collision.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 scale=0.001 0.001 0.001; visual mesh filename=package://fetch_description/meshes/head_box_link.dae scale=0.001 0.001 0.001

Commit message: add fetch-base-camera-mount-mk1 and t265 links to fetch.urdf

File: fetch_description/robots/fetch.urdf (robot description, URDF)
Before this commit: robot fetch, 26 links, 25 joints
Links:
- added link base_camera_mount, mass 70.1294; collision mesh filename=package://jsk_fetch_accessories/base_camera_mount_mk1/fetch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 scale=0.001 0.001 0.001; visual mesh filename=package://jsk_fetch_accessories/base_camera_mount_mk1/fetch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 scale=0.001 0.001 0.001
- added link t265_base_link
Joints:
- added joint base_camera_mount_joint: type fixed, parent base_link, child base_camera_mount, origin xyz=0 0 0 rpy=0 0 0, axis 0 0 1
- added joint t265_to_base_virtual_joint: type fixed, parent t265_base_link, child base_link, origin xyz=0 0 0 rpy=0 0 0, axis 0 0 1
